Commit message: submission1

File: urdf/udacity_bot.xacro (robot description, xacro)
@@ -156,8 +156,15 @@
         </collision>
     </link>
+    <link name="camera_rgbd_frame"></link>
+    <joint name="camera_rgbd_joint" type="fixed">
+        <origin xyz="0 0 0" rpy="-${pi/2} 0 -${pi/2}"/>
+        <parent link="camera"/>
+        <child link="camera_rgbd_frame"/>
+    </joint>
     <joint type="fixed" name="camera_joint">
         <origin xyz="0.25 0 0.2" rpy="0 0 0"/>
         <child link="camera"/>
         <parent link="chassis"/>
+        <axis xyz="0 1 0" rpy="0 0 0"/>
     </joint>
     <link name="camera">
@@ -184,4 +191,5 @@
         <child link="hokuyo"/>
         <parent link="chassis"/>
+        <axis xyz="0 1 0" rpy="0 0 0"/>
     </joint>
     <link name="hokuyo">
